Commit message: t1: make the holosoma 23-DOF mesh-foot URDF the canonical t1.urdf
Replaces the box-foot t1_serial.urdf and the older t1.urdf with the mesh-collision-foot model
(same 23 revolute joints, same names and order; four fixed marker links folded by the importer).
t1/meshes/ now holds that model's export; the 20 meshes only the old URDFs used are dropped.

Claude-Session: https://claude.ai/code/session_01JTwpHNrddHH6F9nd9VmzaY

File: t1/t1.urdf (robot description, URDF)
Before this commit: robot T1, 24 links, 23 joints
Links:
- removed link al1
- removed link al2
- removed link al3
- removed link al4
- removed link ar1
- removed link ar2
- removed link ar3
- removed link ar4
- removed link h1
- removed link h2
- removed link ll1
- removed link ll2
- removed link ll3
- removed link ll4
- removed link ll5
- removed link ll6
- removed link lr1
- removed link lr2
- removed link lr3
- removed link lr4
- removed link lr5
- removed link lr6
- removed link trunk
- removed link waist
- added link AL1, mass 0.53; visual mesh filename=meshes/AL1.STL
- added link AL2, mass 0.160; visual mesh filename=meshes/AL2.STL
- added link AL3, mass 1.02; collision cylinder length=0.15 radius=0.03; visual mesh filename=meshes/AL3.STL
- added link AR1, mass 0.53; visual mesh filename=meshes/AR1.STL
- added link AR2, mass 0.160; visual mesh filename=meshes/AR2.STL
- added link AR3, mass 1.02; collision cylinder length=0.15 radius=0.03; visual mesh filename=meshes/AR3.STL
- added link Ankle_Cross_Left, mass 0.073; visual mesh filename=meshes/Ankle_Cross_Left.STL
- added link Ankle_Cross_Right, mass 0.073; visual mesh filename=meshes/Ankle_Cross_Right.STL
- added link H1, mass 0.443910; visual mesh filename=meshes/H1.STL
- added link H2, mass 0.631019; collision sphere radius=0.08; visual mesh filename=meshes/H2.STL
- added link Hip_Pitch_Left, mass 1.021; visual mesh filename=meshes/Hip_Pitch_Left.STL
- added link Hip_Pitch_Right, mass 1.021; visual mesh filename=meshes/Hip_Pitch_Right.STL
- added link Hip_Roll_Left, mass 0.385; collision cylinder length=0.16 radius=0.05; visual mesh filename=meshes/Hip_Roll_Left.STL
- added link Hip_Roll_Right, mass 0.385; collision cylinder length=0.16 radius=0.05; visual mesh filename=meshes/Hip_Roll_Right.STL
- added link Hip_Yaw_Left, mass 2.166; collision cylinder length=0.08 radius=0.05; visual mesh filename=meshes/Hip_Yaw_Left.STL
- added link Hip_Yaw_Right, mass 2.17; collision cylinder length=0.08 radius=0.05; visual mesh filename=meshes/Hip_Yaw_Right.STL
- added link Shank_Left, mass 1.73; collision box size=0.1 0.08 0.1; visual mesh filename=meshes/Shank_Left.STL
- added link Shank_Right, mass 1.79; collision box size=0.1 0.08 0.1; visual mesh filename=meshes/Shank_Right.STL
- added link Trunk, mass 11.7; collision box size=0.15 0.2 0.3; visual mesh filename=meshes/Trunk.STL
- added link Waist, mass 2.581; visual mesh filename=meshes/Waist.STL
- added link left_foot_contact_point, mass 0.001; visual box size=0.001 0.001 0.001
- added link left_foot_link, mass 0.685; collision mesh filename=meshes/left_foot_link.STL; visual mesh filename=meshes/left_foot_link.STL
- added link left_hand_link, mass 0.327214390850251; collision cylinder length=0.175 radius=0.03; visual mesh filename=meshes/left_hand_link.STL
- added link left_hand_sphere_link, mass 0.001; collision sphere radius=0.005; visual sphere radius=0.005
- added link right_foot_contact_point, mass 0.001; visual box size=0.001 0.001 0.001
- added link right_foot_link, mass 0.685; collision mesh filename=meshes/right_foot_link.STL; visual mesh filename=meshes/right_foot_link.STL
- added link right_hand_link, mass 0.327214390850251; collision cylinder length=0.175 radius=0.03; visual mesh filename=meshes/right_hand_link.STL
- added link right_hand_sphere_link, mass 0.001; collision sphere radius=0.005; visual sphere radius=0.005
Joints:
- removed joint joint_al1
- removed joint joint_al2
- removed joint joint_al3
- removed joint joint_al4
- removed joint joint_ar1
- removed joint joint_ar2
- removed joint joint_ar3
- removed joint joint_ar4
- removed joint joint_h1
- removed joint joint_h2
- removed joint joint_ll1
- removed joint joint_ll2
- removed joint joint_ll3
- removed joint joint_ll4
- removed joint joint_ll5
- removed joint joint_ll6
- removed joint joint_lr1
- removed joint joint_lr2
- removed joint joint_lr3
- removed joint joint_lr4
- removed joint joint_lr5
- removed joint joint_lr6
- removed joint joint_waist
- added joint AAHead_yaw: type revolute, parent Trunk, child H1, origin xyz=0.0625 0 0.243 rpy=0 0 0, axis 0 0 1, limit lower=-1.57 upper=1.57 effort=7 velocity=12.56
- added joint Head_pitch: type revolute, parent H1, child H2, origin xyz=0 0 0.06185 rpy=0 0 0, axis 0 1 0, limit lower=-0.35 upper=1.22 effort=7 velocity=12.56
- added joint Left_Ankle_Pitch: type revolute, parent Shank_Left, child Ankle_Cross_Left, origin xyz=0 0 -0.28 rpy=0 0 0, axis 0 1 0, limit lower=-0.87 upper=0.35 effort=12 velocity=18.8
- added joint Left_Ankle_Roll: type revolute, parent Ankle_Cross_Left, child left_foot_link, origin xyz=0 0.00025 -0.012 rpy=0 0 0, axis 1 0 0, limit lower=-0.44 upper=0.44 effort=12 velocity=12.4
- added joint Left_Elbow_Pitch: type revolute, parent AL2, child AL3, origin xyz=0.00025 0.0605 0 rpy=0 0 0, axis 0 1 0, limit lower=-2.27 upper=2.27 effort=18 velocity=18.84
- added joint Left_Elbow_Yaw: type revolute, parent AL3, child left_hand_link, origin xyz=0 0.1471 0 rpy=0 0 0, axis 0 0 1, limit lower=-2.27 upper=2.27 effort=18 velocity=18.84
- added joint Left_Hip_Pitch: type revolute, parent Waist, child Hip_Pitch_Left, origin xyz=0 0.106 0 rpy=0 0 0, axis 0 1 0, limit lower=-1.8 upper=1.57 effort=45 velocity=12.5
- added joint Left_Hip_Roll: type revolute, parent Hip_Pitch_Left, child Hip_Roll_Left, origin xyz=0 0 -0.02 rpy=0 0 0, axis 1 0 0, limit lower=-0.3 upper=1.57 effort=30 velocity=10.9
- added joint Left_Hip_Yaw: type revolute, parent Hip_Roll_Left, child Hip_Yaw_Left, origin xyz=0 0 -0.081854 rpy=0 0 0, axis 0 0 1, limit lower=-1 upper=1 effort=30 velocity=10.9
- added joint Left_Knee_Pitch: type revolute, parent Hip_Yaw_Left, child Shank_Left, origin xyz=-0.014 0 -0.134 rpy=0 0 0, axis 0 1 0, limit lower=0 upper=2.34 effort=60 velocity=11.7
- added joint Left_Shoulder_Pitch: type revolute, parent Trunk, child AL1, origin xyz=0.0575 0.1063 0.219 rpy=0 0.00088113 0, axis 0 1 0, limit lower=-3.31 upper=1.22 effort=18 velocity=18.84
- added joint Left_Shoulder_Roll: type revolute, parent AL1, child AL2, origin xyz=0 0.047 0 rpy=0 0 0, axis 1 0 0, limit lower=-1.74 upper=1.57 effort=18 velocity=18.84
- added joint Right_Ankle_Pitch: type revolute, parent Shank_Right, child Ankle_Cross_Right, origin xyz=0 0 -0.28 rpy=0 0 0, axis 0 1 0, limit lower=-0.87 upper=0.35 effort=12 velocity=18.8
- added joint Right_Ankle_Roll: type revolute, parent Ankle_Cross_Right, child right_foot_link, origin xyz=0 -0.00025 -0.012 rpy=0 0 0, axis 1 0 0, limit lower=-0.44 upper=0.44 effort=12 velocity=12.4
- added joint Right_Elbow_Pitch: type revolute, parent AR2, child AR3, origin xyz=0.00025 -0.0605 0 rpy=0 0 0, axis 0 1 0, limit lower=-2.27 upper=2.27 effort=18 velocity=18.84
- added joint Right_Elbow_Yaw: type revolute, parent AR3, child right_hand_link, origin xyz=0 -0.1471 0 rpy=0 0 0, axis 0 0 1, limit lower=-2.27 upper=2.27 effort=18 velocity=18.84
- added joint Right_Hip_Pitch: type revolute, parent Waist, child Hip_Pitch_Right, origin xyz=0 -0.106 0 rpy=0 0 0, axis 0 1 0, limit lower=-1.8 upper=1.57 effort=45 velocity=12.5
- added joint Right_Hip_Roll: type revolute, parent Hip_Pitch_Right, child Hip_Roll_Right, origin xyz=0 0 -0.02 rpy=0 0 0, axis 1 0 0, limit lower=-1.57 upper=0.3 effort=30 velocity=10.9
- added joint Right_Hip_Yaw: type revolute, parent Hip_Roll_Right, child Hip_Yaw_Right, origin xyz=0 0 -0.081854 rpy=0 0 0, axis 0 0 1, limit lower=-1 upper=1 effort=30 velocity=10.9
- added joint Right_Knee_Pitch: type revolute, parent Hip_Yaw_Right, child Shank_Right, origin xyz=-0.014 0 -0.134 rpy=0 0 0, axis 0 1 0, limit lower=0 upper=2.34 effort=60 velocity=11.7
- added joint Right_Shoulder_Pitch: type revolute, parent Trunk, child AR1, origin xyz=0.0575 -0.1063 0.219 rpy=0 0.00088113 0, axis 0 1 0, limit lower=-3.31 upper=1.22 effort=18 velocity=18.84
- added joint Right_Shoulder_Roll: type revolute, parent AR1, child AR2, origin xyz=0 -0.047 0 rpy=0 0 0, axis 1 0 0, limit lower=-1.57 upper=1.74 effort=18 velocity=18.84
- added joint Waist: type revolute, parent Trunk, child Waist, origin xyz=0.0625 0 -0.1155 rpy=0 0 0, axis 0 0 1, limit lower=-1.57 upper=1.57 effort=30 velocity=10.88
- added joint left_foot_contact_point: type fixed, parent left_foot_link, child left_foot_contact_point, origin xyz=0 0 -0.032 rpy=0 0 0
- added joint left_hand_sphere_joint: type fixed, parent left_hand_link, child left_hand_sphere_link, origin xyz=0.0 0.2 0.0 rpy=0 0 0
- added joint right_foot_contact_point: type fixed, parent right_foot_link, child right_foot_contact_point, origin xyz=0 0 -0.032 rpy=0 0 0
- added joint right_hand_sphere_joint: type fixed, parent right_hand_link, child right_hand_sphere_link, origin xyz=0.0 -0.2 0.0 rpy=0 0 0

Commit message: t1: knee flexion limit 2.18 rad, the MuJoCo model's range, down from 2.34

File: t1/t1.urdf (robot description, URDF)
Before this commit: robot T1, 28 links, 27 joints
Joints:
- joint Left_Knee_Pitch: limit lower=0 upper=2.34 effort=60 velocity=11.7 -> lower=0 upper=2.18 effort=60 velocity=11.7
- joint Right_Knee_Pitch: limit lower=0 upper=2.34 effort=60 velocity=11.7 -> lower=0 upper=2.18 effort=60 velocity=11.7

Commit message: T1: both shanks 1.82 kg, as Booster's current robot descriptions (booster_assets) give (#4)
Our URDF carried booster_gym's older 1.73 (left) / 1.79 kg (right). booster_assets, Booster's robot-description
repo, has 1.82 kg for both shanks in every T1 model (23/29-dof URDF and MJCF), matching hcrl_sim2real's MJCF; the
inertia tensors and COMs already agree. Lands with the BFM-Zero retrain, since it changes the plant.

File: t1/t1.urdf (robot description, URDF)
Before this commit: robot T1, 28 links, 27 joints
Links:
- link Shank_Left: mass 1.73 -> 1.82
- link Shank_Right: mass 1.79 -> 1.82

Commit message: T1: shank and arm colliders follow the meshes; the shank hull is clipped 0.07-0.23 m below the knee so it clears the thigh and foot, and covers the ball's contact height

File: t1/t1.urdf (robot description, URDF)
Before this commit: robot T1, 28 links, 27 joints
Links:
- link AL3: geometry collision mesh filename=meshes/AL3.STL; visual mesh filename=meshes/AL3.STL
- link AR3: geometry collision mesh filename=meshes/AR3.STL; visual mesh filename=meshes/AR3.STL
- link Shank_Left: geometry collision mesh filename=meshes/collision/Shank_Left.STL; visual mesh filename=meshes/Shank_Left.STL
- link Shank_Right: geometry collision mesh filename=meshes/collision/Shank_Right.STL; visual mesh filename=meshes/Shank_Right.STL
- link left_hand_link: geometry collision mesh filename=meshes/left_hand_link.STL; visual mesh filename=meshes/left_hand_link.STL
- link right_hand_link: geometry collision mesh filename=meshes/right_hand_link.STL; visual mesh filename=meshes/right_hand_link.STL

Commit message: T1: arm and shank collision hulls reduced to 64 vertices (within 4.5 mm of the full hull), so PhysX and Newton collide the same shape

File: t1/t1.urdf (robot description, URDF)
Before this commit: robot T1, 28 links, 27 joints
Links:
- link AL3: geometry collision mesh filename=meshes/collision/AL3.STL; visual mesh filename=meshes/AL3.STL
- link AR3: geometry collision mesh filename=meshes/collision/AR3.STL; visual mesh filename=meshes/AR3.STL
- link left_hand_link: geometry collision mesh filename=meshes/collision/left_hand_link.STL; visual mesh filename=meshes/left_hand_link.STL
- link right_hand_link: geometry collision mesh filename=meshes/collision/right_hand_link.STL; visual mesh filename=meshes/right_hand_link.STL

Commit message: T1: shank and arm colliders are convex decompositions of the meshes (CoACD, 6 pieces per link, 32 vertices each) instead of single hulls; shank pieces clipped 0.07-0.225 m below the knee

File: t1/t1.urdf (robot description, URDF)
Before this commit: robot T1, 28 links, 27 joints
Links:
- link AL3: geometry collision mesh filename=meshes/collision/AL3_0.STL; collision mesh filename=meshes/collision/AL3_1.STL
- link AR3: geometry collision mesh filename=meshes/collision/AR3_0.STL; collision mesh filename=meshes/collision/AR3_1.STL
- link Shank_Left: geometry collision mesh filename=meshes/collision/Shank_Left_0.STL; collision mesh filename=meshes/collision/Shank_Left_1.STL
- link Shank_Right: geometry collision mesh filename=meshes/collision/Shank_Right_0.STL; collision mesh filename=meshes/collision/Shank_Right_1.STL
- link left_hand_link: geometry collision mesh filename=meshes/collision/left_hand_link_0.STL; collision mesh filename=meshes/collision/left_hand_link_1.STL
- link right_hand_link: geometry collision mesh filename=meshes/collision/right_hand_link_0.STL; collision mesh filename=meshes/collision/right_hand_link_1.STL

Commit message: T1 collision pieces: the right side mirrors the left (y -> -y), every piece capped at 32 vertices; shanks 5 pieces, arm links 6

File: t1/t1.urdf (robot description, URDF)
Before this commit: robot T1, 28 links, 27 joints
Links:
- link Shank_Right: geometry collision mesh filename=meshes/collision/Shank_Right_0.STL; collision mesh filename=meshes/collision/Shank_Right_1.STL

Commit message: T1 colliders: the feet are convex decompositions too (8 pieces, sole unchanged), freeing the shank to reach 0.25 m below the knee (13 pieces); the foot's front piece is chamfered ahead of the ankle so the shin clears it over the whole ankle range

File: t1/t1.urdf (robot description, URDF)
Before this commit: robot T1, 28 links, 27 joints
Links:
- link Shank_Left: geometry collision mesh filename=meshes/collision/Shank_Left_0.STL; collision mesh filename=meshes/collision/Shank_Left_1.STL
- link Shank_Right: geometry collision mesh filename=meshes/collision/Shank_Right_0.STL; collision mesh filename=meshes/collision/Shank_Right_1.STL
- link left_foot_link: geometry collision mesh filename=meshes/collision/left_foot_link_0.STL; collision mesh filename=meshes/collision/left_foot_link_1.STL
- link right_foot_link: geometry collision mesh filename=meshes/collision/right_foot_link_0.STL; collision mesh filename=meshes/collision/right_foot_link_1.STL

Commit message: T1 colliders: shank and foot collide on their own meshes (one convex hull each); only the upper arms and forearms are decompositions (6 pieces, 64 vertices); the shank-foot and knee pairs are filtered in the simulators

File: t1/t1.urdf (robot description, URDF)
Before this commit: robot T1, 28 links, 27 joints
Links:
- link Shank_Left: geometry collision mesh filename=meshes/Shank_Left.STL; visual mesh filename=meshes/Shank_Left.STL
- link Shank_Right: geometry collision mesh filename=meshes/Shank_Right.STL; visual mesh filename=meshes/Shank_Right.STL
- link left_foot_link: geometry collision mesh filename=meshes/left_foot_link.STL; visual mesh filename=meshes/left_foot_link.STL
- link right_foot_link: geometry collision mesh filename=meshes/right_foot_link.STL; visual mesh filename=meshes/right_foot_link.STL

Commit message: T1: shank and arm colliders follow the meshes (#5)
* T1: shank and arm colliders follow the meshes; the shank hull is clipped 0.07-0.23 m below the knee so it clears the thigh and foot, and covers the ball's contact height

* T1: arm and shank collision hulls reduced to 64 vertices (within 4.5 mm of the full hull), so PhysX and Newton collide the same shape

* T1: shank and arm colliders are convex decompositions of the meshes (CoACD, 6 pieces per link, 32 vertices each) instead of single hulls; shank pieces clipped 0.07-0.225 m below the knee

* T1 collision pieces: the right side mirrors the left (y -> -y), every piece capped at 32 vertices; shanks 5 pieces, arm links 6

* T1 colliders: the feet are convex decompositions too (8 pieces, sole unchanged), freeing the shank to reach 0.25 m below the knee (13 pieces); the foot's front piece is chamfered ahead of the ankle so the shin clears it over the whole ankle range

* T1 colliders: shank and foot collide on their own meshes (one convex hull each); only the upper arms and forearms are decompositions (6 pieces, 64 vertices); the shank-foot and knee pairs are filtered in the simulators

File: t1/t1.urdf (robot description, URDF)
Before this commit: robot T1, 28 links, 27 joints
Links:
- link AL3: geometry collision mesh filename=meshes/collision/AL3_0.STL; collision mesh filename=meshes/collision/AL3_1.STL
- link AR3: geometry collision mesh filename=meshes/collision/AR3_0.STL; collision mesh filename=meshes/collision/AR3_1.STL
- link Shank_Left: geometry collision mesh filename=meshes/Shank_Left.STL; visual mesh filename=meshes/Shank_Left.STL
- link Shank_Right: geometry collision mesh filename=meshes/Shank_Right.STL; visual mesh filename=meshes/Shank_Right.STL
- link left_hand_link: geometry collision mesh filename=meshes/collision/left_hand_link_0.STL; collision mesh filename=meshes/collision/left_hand_link_1.STL
- link right_hand_link: geometry collision mesh filename=meshes/collision/right_hand_link_0.STL; collision mesh filename=meshes/collision/right_hand_link_1.STL
